File: hardware/uartdbg_232/uartdbg_232/uartdbg_232.kicad_pcb (KiCad board)
At the start: 2 copper layers, 40 x 30.5 mm, 10 parts, among them J1 Conn_01x04_Female, J2 Conn_01x06_Female, J3 DB9_Female, U1 MAX232

Commit message: [CHG][NT] 暂存
Parts:
- added SYM2: SYM_Magnet_Small, Symbol:OSHW-Logo2_7.3x6mm_Copper, F.Cu at (124.0, 94.3)
- C1, C2, C3, C4, C5: footprint Capacitor_SMD:C_0603_1608Metric_Pad1.08x0.95mm_HandSolder -> Red_Pro:C_0603_1608Metric_Pad1.08x0.95mm_HandSolder
- J3: footprint Connector_Dsub:DSUB-9_Female_Horizontal_P2.77x2.84mm_EdgePinOffset7.70mm_Housed_MountingHolesOffset9.12mm -> Red_Pro:DSUB-9_Female_Horizontal_P2.77x2.84mm_EdgePinOffset7.70mm_Housed_MountingHolesOffset9.12mm
- moved SYM1 1.03 mm to (110.0, 95.8)
Routing:
- net /RS232_TX: track 0.00 -> 22.2 mm
- net +5V: track 0.00 -> 16.7 mm, vias 0 -> 1
- net /RS232_RX: track 0.00 -> 15.3 mm
- net /TTL_RX: track 0.00 -> 10.9 mm
- net /TTL_TX: track 0.00 -> 10.2 mm
- net GND: track 0.00 -> 9.87 mm, vias 0 -> 1
- net Net-(C4-Pad2): track 0.00 -> 3.71 mm, vias 0 -> 1
- net Net-(C5-Pad2): track 0.00 -> 3.41 mm, vias 0 -> 1
- net Net-(C3-Pad2): track 0.00 -> 3.34 mm, vias 0 -> 1
- net Net-(C3-Pad1): track 0.00 -> 3.14 mm, vias 0 -> 1
- net Net-(C1-Pad2): track 0.00 -> 2.62 mm
- net Net-(C1-Pad1): track 0.00 -> 2.34 mm
Other:
- net class Default: trace_width 0.25 -> 0.2; via_dia 0.8 -> 0.6; via_drill 0.4 -> 0.3
- net class power added: clearance 0.2, trace_width 0.3, via_dia 0.8, via_drill 0.4
- net class power5v added: clearance 0.2, trace_width 0.5, via_dia 0.8, via_drill 0.5
- board text added: "GND TX RX 5V"
